File: arduino-mega-isa-shield.kicad_pcb (KiCad board)
At the start: 2 copper layers, 144.7 x 80.3 mm, 11 parts, among them J1 EBC49DCWN-S420, J2 JST VH 1x6, U1 501MILFT, Y1 3.579545MHZ

Commit message: Reverse LA17-LA23 for sequential port access, re-route board
Parts:
- U1: value 501MILFT -> ICS501
Connections:
- XA1 pad A10: /LA21 -> /LA19
- XA1 pad A12: /LA19 -> /LA21
- XA1 pad A13: /LA18 -> /LA22
- XA1 pad A14: /LA17 -> /LA23
- XA1 pad A8: /LA23 -> /LA17
- XA1 pad A9: /LA22 -> /LA18
Routing:
- net /OSC_14M318: track 65.2 -> 153.9 mm, vias 2 -> 0
- net /A1: track 116.7 -> 70.8 mm
- net /LA18: track 63.4 -> 100.9 mm, vias 0 -> 1
- net /LA22: track 63.4 -> 95.4 mm, vias 0 -> 1
- net /LA17: track 63.9 -> 94.6 mm, vias 0 -> 1
- net /DRQ1: track 112.2 -> 141.2 mm
- net /PH3: track 54.6 -> 80.2 mm, vias 1 -> 0
- net /LA20: track 63.4 -> 88.5 mm, vias 0 -> 1
- net /A8: track 75.2 -> 99.6 mm, vias 0 -> 1
- net /PG1: track 130.5 -> 108.8 mm
- net /A11: track 75.5 -> 96.2 mm
- net /LA21: track 63.4 -> 82.7 mm, vias 0 -> 1
- net /A9: track 94.2 -> 75.2 mm
- net /A3: track 92.6 -> 75.4 mm, vias 1 -> 0
- net /PG2: track 109.2 -> 126.2 mm, vias 2 -> 1
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
Commit message: Update board for EDAC 395-098-520-350 ISA connector
Parts:
- J1: value EBC49DCWN-S420 -> 395-098-520-350
Changed lines of the file:
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@@
     (fp_line (start -0.254 -31.9396) (end -6.594 -31.9396) (layer "B.CrtYd") (width 0.15))
     (fp_line (start -1.934 -12.5476) (end -1.934 -3.0486) (layer "B.CrtYd") (width 0.15))
-    (fp_arc (start 99.8728 -1.7018) (mid 99.650928 -1.077973) (end 99.314 -0.508) (layer "B.CrtYd") (width 0.15))
+    (fp_arc (start 99.8728 -1.7018) (mid 99.650934 -1.077968) (end 99.314 -0.508) (layer "B.CrtYd") (width 0.15))
     (fp_arc (start 98.552 0.254) (mid 96.52 0.914237) (end 94.488 0.254) (layer "B.CrtYd") (width 0.15))
     (fp_arc (start 88.138 -53.594) (mid 90.17 -54.254237) (end 92.202 -53.594) (layer "B.CrtYd") (width 0.15))
@@
       (effects (font (size 1 1) (thickness 0.15)))
     )
-    (fp_text value "EBC49DCWN-S420" (at -64.77 2.54) (layer "F.SilkS")
-      (effects (font (size 1 1) (thickness 0.15)))
-    )
+    (fp_text value "395-098-520-350" (at -64.77 2.54) (layer "F.SilkS")
+      (effects (font (size 1 1) (thickness 0.15)))
+    )
